File: KiCAD_Proj/PowerManagement.kicad_sch (KiCad schematic)
At the start: 23 parts, among them IC3 TPS51397ARJER, J1 691401700003B

Commit message: Schematic nearly done, ordened
Parts:
- removed J1: 691401700003B, SamacSys_Parts:691401700003B, symbol Healthbot-Symbols:Terminal_Block3
- removed PS1: TSR_1-2433, SamacSys_Parts:TSR-1-2433, symbol Healthbot-Symbols:DC-DC_3.3V
- added TP1: ~, TestPoint:TestPoint_Pad_D1.5mm, symbol Connector:TestPoint
Connections:
- net +12V: no longer C10.2, C11.2, C12.2, C13.2, C14.2, C4.1, C5.1, C5.2, C6.1, C6.2, C7.1, C7.2, IC3.10 (NC_1), IC3.13 (AGND), IC3.16 (NC_2), IC3.18 (PGND_3), IC3.2 (VIN_1), IC3.21 (PGND_4), IC3.3 (VIN_2), IC3.4 (VIN_3), IC3.5 (VIN_4), IC3.7 (PGND_1), IC3.8 (PGND_2), R14.2, R17.2
- net FB: now also TP1.1
- net +5V renamed 5V
- new net GND: C10.2, C11.2, C12.2, C13.2, C14.2, C4.1, C5.1, C5.2, C6.1, C6.2, C7.1, C7.2, IC3.10 (NC_1), IC3.13 (AGND), IC3.16 (NC_2), IC3.18 (PGND_3), IC3.2 (VIN_1), IC3.21 (PGND_4), IC3.3 (VIN_2), IC3.4 (VIN_3), IC3.5 (VIN_4), IC3.7 (PGND_1), IC3.8 (PGND_2), R14.2, R17.2
Other:
- moved on the sheet: C10, C11, C12, C13, C14, C4, C5, C6, C7, C8, C9, IC3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

Commit message: Finished schematic, in review
Connections:
- no-connect marks 0 -> 1
Other:
- company: (none) -> HAN Univeristy of Applied Sciences
- title: (none) -> Project_Healthbot_HAT
Changed lines of the file:
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@@
 (kicad_sch (version 20230121) (generator eeschema)
   (paper "A4")
+  (title_block
+    (title "Project_Healthbot_HAT")
+    (date "2024-05-16")
+    (rev "V0.1")
+    (company "HAN Univeristy of Applied Sciences")
+    (comment 1 "Marelle Vink")
+  )
   (junction (at 229.87 95.25) (diameter 0) (color 0 0 0 0)
   )
@@
   (junction (at 83.82 99.06) (diameter 0) (color 0 0 0 0)
   )
+  (no_connect (at 119.38 99.06))
   (wire (pts (xy 172.72 102.87) (xy 172.72 107.95))
     (stroke (width 0) (type default))

Commit message: -add missing connections in schematic, and some other small changes
Connections:
- net GND: now also C4.2; no longer C4.1
- net VCC: now also C4.1; no longer C4.2
Other:
- moved on the sheet: C4

Commit message: Schematic finished
Parts:
- removed L1: 1.8uH, Inductor_SMD:L_0603_1608Metric_Pad1.05x0.95mm_HandSolder, symbol Device:L
- added L1: SRP6540-1R0M, INDPM7265X400N, symbol Healthbot-Symbols:SRP6540-1R0M
Connections:
- net 5V: now also L1.2
- net SW: now also L1.1
Other:
- moved on the sheet: C4

Commit message: All components placed
Parts:
- removed TP1: ~, TestPoint:TestPoint_Pad_D1.5mm, symbol Connector:TestPoint
Connections:
- net GND: no longer C5.1, C6.1, C7.1, IC3.2 (VIN_1), IC3.3 (VIN_2), IC3.4 (VIN_3), IC3.5 (VIN_4)
- new net 12V: C5.1, C6.1, C7.1, IC3.2 (VIN_1), IC3.3 (VIN_2), IC3.4 (VIN_3), IC3.5 (VIN_4)
Changed lines of the file:
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@@
-	)
-	(junction
-		(at 71.12 99.06)
-		(diameter 0)
-		(color 0 0 0 0)
 	)
 	(junction
@@
 	)
 	(junction
-		(at 172.72 102.87)
-		(diameter 0)
-		(color 0 0 0 0)
-	)
-	(junction
 		(at 60.96 99.06)
 		(diameter 0)
@@
 	)
 	(junction
-		(at 83.82 99.06)
-		(diameter 0)
-		(color 0 0 0 0)
-	)
-	(junction
 		(at 171.45 95.25)
 		(diameter 0)
@@
 		(pts
 			(xy 83.82 99.06) (xy 88.9 99.06)
-		)
-		(stroke
-			(width 0)
-			(type default)
-		)
-	)
-	(wire
-		(pts
-			(xy 71.12 99.06) (xy 83.82 99.06)
 		)
 		(stroke
@@
 					(unit 1)
 				)
-			)
-		)
-	)
-	(symbol
-		(lib_id "Connector:TestPoint")
-		(at 172.72 102.87 0)
-		(unit 1)
-		(exclude_from_sim no)
-		(in_bom yes)
-		(on_board yes)
-		(dnp no)
-		(property "Reference" "TP1"
-			(at 173.99 99.06 0)
-			(effects
-				(font
-					(size 1.27 1.27)
-				)
-				(justify left)
-			)
-		)
-		(property "Value" "~"
-			(at 173.99 100.33 0)
-			(effects
-				(font
-					(size 1.27 1.27)
-				)
-				(justify left)
-			)
-		)
-		(property "Footprint" "TestPoint:TestPoint_Pad_D1.5mm"
-			(at 177.8 102.87 0)
-			(effects
-				(font
-					(size 1.27 1.27)
-				)
-				(hide yes)
-			)
-		)
-		(property "Datasheet" "~"
-			(at 177.8 102.87 0)
-			(effects
-				(font
-					(size 1.27 1.27)
-				)
-				(hide yes)
-			)
-		)
-		(property "Description" ""
-			(at 172.72 102.87 0)
-			(effects
-				(font
-					(size 1.27 1.27)
-				)
-				(hide yes)
-			)
-		)
-		(pin "1"
-		)
-		(instances
-			(project "universalConnectorBoard"
-				(path "/4d36baa7-ef48-416a-b1c8-6a662c0af28f/26655477-e6dc-458e-ab5c-3170a4e00944"
-					(reference "TP1")
-					(unit 1)
-				)

Commit message: PCB Design halfway
Connections:
- net +12V renamed +3.3V
Changed lines of the file:
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@@
+	)
+	(symbol
+		(lib_id "power:+3.3V")
+		(at 133.35 99.06 0)
+		(unit 1)
+		(exclude_from_sim no)
+		(in_bom yes)
+		(on_board yes)
+		(dnp no)
+		(property "Reference" "#PWR027"
+			(at 133.35 102.87 0)
+			(effects
+				(font
+					(size 1.27 1.27)
+				)
+				(hide yes)
+			)
+		)
+		(property "Value" "+3.3V"
+			(at 133.35 94.996 0)
+			(effects
+				(font
+					(size 1.27 1.27)
+				)
+			)
+		)
+		(property "Footprint" ""
+			(at 133.35 99.06 0)
+			(effects
+				(font
+					(size 1.27 1.27)
+				)
+				(hide yes)
+			)
+		)
+		(property "Datasheet" ""
+			(at 133.35 99.06 0)
+			(effects
+				(font
+					(size 1.27 1.27)
+				)
+				(hide yes)
+			)
+		)
+		(property "Description" "Power symbol creates a global label with name \"+3.3V\""
+			(at 133.35 99.06 0)
+			(effects
+				(font
+					(size 1.27 1.27)
+				)
+				(hide yes)
+			)
+		)
+		(pin "1"
+		)
+		(instances
+			(project "universalConnectorBoard"
+				(path "/4d36baa7-ef48-416a-b1c8-6a662c0af28f/26655477-e6dc-458e-ab5c-3170a4e00944"
+					(reference "#PWR027")
+					(unit 1)
+				)
+			)
+		)
 	)
 	(symbol
@@
 					(unit 1)
 				)
-			)
-		)
-	)
-	(symbol
-		(lib_id "power:+12V")
-		(at 133.35 99.06 0)
-		(unit 1)
-		(exclude_from_sim no)
-		(in_bom yes)
-		(on_board yes)
-		(dnp no)
-		(property "Reference" "#PWR060"
-			(at 133.35 102.87 0)
-			(effects
-				(font
-					(size 1.27 1.27)
-				)
-				(hide yes)
-			)
-		)
-		(property "Value" "+12V"
-			(at 133.35 94.996 0)
-			(effects
-				(font
-					(size 1.27 1.27)
-				)
-			)
-		)
-		(property "Footprint" ""
-			(at 133.35 99.06 0)
-			(effects
-				(font
-					(size 1.27 1.27)
-				)
-				(hide yes)
-			)
-		)
-		(property "Datasheet" ""
-			(at 133.35 99.06 0)
-			(effects
-				(font
-					(size 1.27 1.27)
-				)
-				(hide yes)
-			)
-		)
-		(property "Description" "Power symbol creates a global label with name \"+12V\""
-			(at 133.35 99.06 0)
-			(effects
-				(font
-					(size 1.27 1.27)
-				)
-				(hide yes)
-			)
-		)
-		(pin "1"
-		)
-		(instances
-			(project "universalConnectorBoard"
-				(path "/4d36baa7-ef48-416a-b1c8-6a662c0af28f/26655477-e6dc-458e-ab5c-3170a4e00944"
-					(reference "#PWR060")
-					(unit 1)
-				)

Commit message: Finished!
Parts:
- L1: footprint INDPM7265X400N -> Healthbot-Footprints:INDPM7265X400N
Changed lines of the file:
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@@
 			)
 		)
-		(property "Footprint" "INDPM7265X400N"
+		(property "Footprint" "Healthbot-Footprints:INDPM7265X400N"
 			(at 193.04 191.44 0)
 			(effects
