File: KiCAD_Proj/universalConnectorBoard.kicad_pcb (KiCad board)
At the start: 2 copper layers, 65 x 56.5 mm, 92 parts, among them IC1 RPI_Pico_EvaluationBoard, IC2 SN74LV4052ADR, IC3 TPS51397ARJER, IC4 TCA9534DWR, J1 691401700003B, J10 Cheeks, J11 MD_SW1, J12 MD_SW2, J13 Motor1, J14 Motor2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

Commit message: Schematic finished
Parts:
- added C15: Elec_Capacitor, SamacSys_Parts:CAPAE1000X1050N, F.Cu at (44.3, 62.9)
- added C17: Elec_Capacitor, SamacSys_Parts:CAPAE1000X1050N, F.Cu at (44.3, 74.9)
- added C22: 100nF, Capacitor_SMD:C_0603_1608Metric_Pad1.08x0.95mm_HandSolder, F.Cu at (47.1, 34.5)
- added J15: Extra VCC/GND, Connector_PinHeader_2.54mm:PinHeader_2x03_P2.54mm_Vertical, F.Cu at (56.5, 69.4)
- added L1: SRP6540-1R0M, Healthbot-Footprints:INDPM7265X400N, F.Cu at (59.2, 61.0)
- added R31: 4.7k, Resistor_SMD:R_0603_1608Metric_Pad0.98x0.95mm_HandSolder, F.Cu at (47.1, 37.0)
- added U3: RASPBERRY_PI_4B_4GB, RASPBERRY_PI_4B_4GB:MODULE_RASPBERRY_PI_4B_4GB, F.Cu at (56.8, 126.0)
- C16, C18: footprint Capacitor_SMD:C_0805_2012Metric_Pad1.18x1.45mm_HandSolder -> Capacitor_SMD:C_0603_1608Metric_Pad1.08x0.95mm_HandSolder
Connections:
- C16 pad 1: /StepperMotors/3.3V+ -> +3.3V
- C18 pad 1: /StepperMotors/3.3V+ -> +3.3V
- C21 pad 1: GND -> +12V
- C4 pad 1: +12V -> /Regulator5V/VCC
- C4 pad 2: /Regulator5V/VCC -> +12V
- IC1 pad 10: /MUX_B -> /Display_RES
- IC1 pad 14: /Display_SDA -> /Display_CLK
- IC1 pad 15: /Display_SCL -> /Display_MOSI
- IC1 pad 16: /Display_RES -> /Radar_MISO
- IC1 pad 33: unconnected-(IC1-AGND-Pad33) -> GND
- IC1 pad 9: /MUX_A -> /Radar_INT
- IC2 pad 11: /MUX_RX4 -> /MUX_TX4
- IC4 pad 11: /MUX_GPIO6 -> /MUX_B
- IC4 pad 12: /MUX_GPIO7 -> /MUX_A
- J1 pad 4: GND -> +12V
- J6 pad 3: /MUX_RX4 -> /MUX_TX4
- JP2 pad 1: /StepperMotors/3.3V+ -> +3.3V
- JP3 pad 1: /StepperMotors/3.3V+ -> +3.3V
- JP4 pad 1: /StepperMotors/3.3V+ -> +3.3V
- JP5 pad 1: /StepperMotors/3.3V+ -> +3.3V
- PS1 pad 2: GND -> +12V
- R22 pad 1: /LED_Cheeks -> Net-(Q2-G)
- R22 pad 2: Net-(Q2-G) -> /LED_Cheeks
- R26 pad 1: /LED_Mouth -> Net-(Q1-G)
- R26 pad 2: Net-(Q1-G) -> /LED_Mouth
- R4 pad 2: /MUX_RX4 -> /MUX_TX4
- SW1 pad 1: GND -> Net-(R31-Pad2)

Commit message: Added Pi HAT reference footprint
Parts:
- removed the C15 at (139.7, 73.7)
- removed the C15 at (44.3, 62.9)
- removed the C17 at (152.4, 73.7)
- removed the C17 at (44.3, 74.9)
- removed the L1 at (59.2, 61.0)
- removed the L1 at (171.1, 137.2)
- removed the R22 at (206.6, 137.2)
- removed the R22 at (147.6, 133.6)
- removed the R23 at (145.1, 133.6)
- removed the R23 at (206.6, 139.7)
- removed REF** (x4): MountingHole_2.7mm_M2.5, MountingHole:MountingHole_2.7mm_M2.5
- added C15: Elec_Capacitor, SamacSys_Parts:CAPAE1000X1050N, F.Cu at (226.8, 80.8)
- added C17: Elec_Capacitor, SamacSys_Parts:CAPAE1000X1050N, F.Cu at (226.8, 92.9)
- added L1: SRP6540-1R0M, Healthbot-Footprints:INDPM7265X400N, F.Cu at (237.0, 116.0)
- added R22: 47, Resistor_SMD:R_0603_1608Metric_Pad0.98x0.95mm_HandSolder, F.Cu at (183.5, 118.4)
- added R23: 50k, Resistor_SMD:R_0603_1608Metric_Pad0.98x0.95mm_HandSolder, F.Cu at (183.5, 121.0)
- J7: value Extra GPIO output -> Radar; footprint Connector_PinHeader_2.54mm:PinHeader_1x02_P2.54mm_Vertical -> Connector_JST:JST_XH_S8B-XH-A_1x08_P2.50mm_Horizontal
- U1, U2: footprint TMC2209_SILENTSTEPSTICK:MODULE_TMC2209_SILENTSTEPSTICK -> Healthbot-Footprints:MODULE_TMC2209_SILENTSTEPSTICK
- U3: footprint RASPBERRY_PI_4B_4GB:MODULE_RASPBERRY_PI_4B_4GB -> Healthbot-Footprints:MODULE_RASPBERRY_PI_4B_4GB
- moved J4 183.2 mm to (38.2, 66.2)
- moved R31 163.9 mm to (187.9, 121.0)
- moved C22 155.7 mm to (174.8, 123.5)
- moved J15 154.9 mm to (211.4, 69.1)
- moved U2 107.5 mm to (245.1, 63.9)
- moved Q1 100.8 mm to (211.5, 55.3), turned to 0 degrees
- moved JP2 99.8 mm to (236.8, 76.6), turned to 0 degrees
- moved Q2 99.7 mm to (211.5, 60.0), turned to 0 degrees
- moved Q3 99.0 mm to (211.5, 64.6), turned to 0 degrees
- moved J2 97.9 mm to (190.6, 56.3)
- moved JP3 95.9 mm to (236.8, 80.1), turned to 0 degrees
- moved C18 90.3 mm to (236.8, 92.8), turned to 0 degrees
- moved JP7 87.2 mm to (201.7, 125.6), turned to 0 degrees
- moved JP4 82.6 mm to (236.8, 83.7), turned to 0 degrees
- moved JP6 82.0 mm to (197.0, 125.6), turned to 0 degrees
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Connections:
- J7 pad 1: /MUX_GPIO6 -> /Radar_RES
- J7 pad 2: /MUX_GPIO7 -> /Radar_CS
- U1 pad 2: /StepperMotors/3.3V+ -> +3.3V
- U1 pad 8: /StepperMotors/12V+ -> +12V
- U2 pad 2: /StepperMotors/3.3V+ -> +3.3V
- U2 pad 8: /StepperMotors/12V+ -> +12V
- U3 pad 1: Net-(U3-3V3-Pad1) -> unconnected-(U3-3V3-Pad1)
- U3 pad 14: Net-(U3-GND-Pad14) -> unconnected-(U3-GND-Pad14)_4
- U3 pad 17: Net-(U3-3V3-Pad1) -> unconnected-(U3-3V3-Pad1)_0
- U3 pad 2: Net-(U3-5V-Pad2) -> unconnected-(U3-5V-Pad2)
- U3 pad 20: Net-(U3-GND-Pad14) -> unconnected-(U3-GND-Pad14)_6
- U3 pad 25: Net-(U3-GND-Pad14) -> unconnected-(U3-GND-Pad14)_3
- U3 pad 30: Net-(U3-GND-Pad14) -> unconnected-(U3-GND-Pad14)_0
- U3 pad 34: Net-(U3-GND-Pad14) -> unconnected-(U3-GND-Pad14)_1
- U3 pad 39: Net-(U3-GND-Pad14) -> unconnected-(U3-GND-Pad14)_2
- U3 pad 4: Net-(U3-5V-Pad2) -> unconnected-(U3-5V-Pad2)_0
- U3 pad 6: Net-(U3-GND-Pad14) -> unconnected-(U3-GND-Pad14)_5
- U3 pad 9: Net-(U3-GND-Pad14) -> unconnected-(U3-GND-Pad14)
- U3 pad S1: Net-(U3-SHIELD-PadS1) -> unconnected-(U3-SHIELD-PadS1)_1
- U3 pad S2: Net-(U3-SHIELD-PadS1) -> unconnected-(U3-SHIELD-PadS1)_2
- U3 pad S3: Net-(U3-SHIELD-PadS1) -> unconnected-(U3-SHIELD-PadS1)
- U3 pad S4: Net-(U3-SHIELD-PadS1) -> unconnected-(U3-SHIELD-PadS1)_0
Other:
- board outline removed

Commit message: All components placed
Parts:
- removed J4: RPI4, Connector_PinHeader_2.54mm:PinHeader_2x20_P2.54mm_Vertical
- removed TP1: ~, TestPoint:TestPoint_Pad_D1.5mm
- added TP10: TP_VCC_MUX, TestPoint:TestPoint_Pad_D1.5mm, F.Cu at (269.3, 82.9)
- added TP11: TP_VSYS, TestPoint:TestPoint_Pad_D1.5mm, F.Cu at (269.3, 86.5)
- added TP12: TP_VCC_LEDM, TestPoint:TestPoint_Pad_D1.5mm, F.Cu at (264.3, 72.1)
- added TP13: TP_VCC_LEDC, TestPoint:TestPoint_Pad_D1.5mm, F.Cu at (264.3, 75.7)
- added TP14: TP_GND, TestPoint:TestPoint_Pad_D1.5mm, F.Cu at (272.9, 79.4)
- added TP15: TP_5V_RPI4, TestPoint:TestPoint_Pad_D1.5mm, F.Cu at (272.9, 82.9)
- added TP2: TP_3.3V, TestPoint:TestPoint_Pad_D1.5mm, B.Cu at (89.9, 58.2)
- added TP3: TP_12V, TestPoint:TestPoint_Pad_D1.5mm, F.Cu at (129.8, 55.4)
- added TP4: TP_5V, TestPoint:TestPoint_Pad_D1.5mm, B.Cu at (89.9, 64.3)
- added TP5: TP_GND, TestPoint:TestPoint_Pad_D1.5mm, F.Cu at (265.8, 82.9)
- added TP6: TP_RX, TestPoint:TestPoint_Pad_D1.5mm, F.Cu at (265.8, 86.5)
- added TP7: TP_TX, TestPoint:TestPoint_Pad_D1.5mm, F.Cu at (269.3, 72.3)
- added TP8: TP_VCC_STRIP1, TestPoint:TestPoint_Pad_D1.5mm, F.Cu at (269.3, 75.8)
- added TP9: TP_VCC_STRIP2, TestPoint:TestPoint_Pad_D1.5mm, F.Cu at (269.3, 79.4)
- JP6: value Ledstrip_VCC -> Ledstrip1_VCC
- JP7: value Ledstrip_VCC -> Ledstrip2_VCC
- PS1: footprint SamacSys_Parts:TSR-1-2433 -> Healthbot-Footprints:TSR-1-2433
- R24: value 50k -> 75
- R26: value 47 -> 50k
- R29: value 75 -> 47
- moved J3 140.1 mm to (56.9, 111.9), turned to -90 degrees
- moved C16 138.8 mm to (100.1, 113.9), turned to -90 degrees
- moved Q3 137.9 mm to (80.4, 107.5)
- moved C18 137.8 mm to (100.1, 109.4), turned to -90 degrees
- moved L1 136.8 mm to (111.0, 62.6), turned to 90 degrees
- moved J2 133.8 mm to (56.8, 55.7), turned to -90 degrees
- moved J8 133.1 mm to (63.7, 127.5)
- moved PS1 132.3 mm to (98.2, 59.6), turned to -90 degrees
- moved JP6 131.3 mm to (65.9, 118.6), turned to 90 degrees
- moved C14 128.7 mm to (109.3, 54.1), turned to -90 degrees
- moved U1 126.4 mm to (110.5, 111.0)
- moved C13 126.2 mm to (110.9, 54.1), turned to -90 degrees
- moved JP2 124.5 mm to (120.3, 120.1), turned to 180 degrees
- moved U2 124.2 mm to (130.3, 111.3)
- moved JP7 124.1 mm to (77.8, 118.6), turned to 90 degrees
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Connections:
- C10 pad 2: +12V -> GND
- C11 pad 2: +12V -> GND
- C12 pad 2: +12V -> GND
- C13 pad 2: +12V -> GND
- C14 pad 2: +12V -> GND
- C21 pad 1: +12V -> GND
- C4 pad 2: +12V -> GND
- C5 pad 2: +12V -> GND
- C6 pad 2: +12V -> GND
- C7 pad 2: +12V -> GND
- IC1 pad 19: /MUX_INH -> /Ledstrip1_DATA
- IC1 pad 20: /Ledstrip1_DATA -> /Ledstrip2_DATA
- IC1 pad 21: /Ledstrip2_DATA -> /MUX_INH
- IC3 pad 10: +12V -> GND
- IC3 pad 13: +12V -> GND
- IC3 pad 16: +12V -> GND
- IC3 pad 18: +12V -> GND
- IC3 pad 21: +12V -> GND
- IC3 pad 7: +12V -> GND
- IC3 pad 8: +12V -> GND
- J1 pad 4: +12V -> GND
- PS1 pad 2: +12V -> GND
- R14 pad 2: +12V -> GND
- R17 pad 2: +12V -> GND
- R24 pad 1: +3.3V -> Net-(J10-Pin_2)
- R26 pad 1: Net-(Q1-G) -> +3.3V
- R26 pad 2: /LED_Mouth -> GND
- R29 pad 1: Net-(J10-Pin_2) -> Net-(Q1-G)
- R29 pad 2: GND -> /LED_Mouth
- SW1 pad 2: Net-(J4-Pin_36) -> Net-(U3-GPIO16)
- U3 pad 10: unconnected-(U3-GPIO15/RXD0-Pad10) -> /RXD_PI4
- U3 pad 14: unconnected-(U3-GND-Pad14)_4 -> GND
- U3 pad 15: unconnected-(U3-GPIO22/GPIO_GEN3-Pad15) -> /SWDIO
- U3 pad 18: unconnected-(U3-GPIO24/GPIO_GEN5-Pad18) -> /SWCLK
- U3 pad 2: unconnected-(U3-5V-Pad2) -> +5V
- U3 pad 20: unconnected-(U3-GND-Pad14)_6 -> GND
- U3 pad 25: unconnected-(U3-GND-Pad14)_3 -> GND
- U3 pad 30: unconnected-(U3-GND-Pad14)_0 -> GND
- U3 pad 34: unconnected-(U3-GND-Pad14)_1 -> GND
- U3 pad 36: unconnected-(U3-GPIO16-Pad36) -> Net-(U3-GPIO16)
- U3 pad 39: unconnected-(U3-GND-Pad14)_2 -> GND
- U3 pad 4: unconnected-(U3-5V-Pad2)_0 -> +5V
- U3 pad 6: unconnected-(U3-GND-Pad14)_5 -> GND
- U3 pad 8: unconnected-(U3-GPIO14/TXD0-Pad8) -> /TXD_PI4
- U3 pad 9: unconnected-(U3-GND-Pad14) -> GND
Other:
- board outline added: 113.2 x 85 mm
- board text added: "CAMERA"

Commit message: Minor movements
Parts:
- TP3, TP7: moved to B.Cu
- moved TP7 220.2 mm to (51.8, 106.6), turned to 180 degrees
- moved TP6 217.8 mm to (48.9, 106.6)
- moved TP8 208.1 mm to (64.9, 114.7)
- moved TP11 205.0 mm to (64.6, 74.0)
- moved C19 200.7 mm to (67.9, 111.6)
- moved C2 198.8 mm to (68.2, 122.8)
- moved TP9 195.3 mm to (77.2, 114.7)
- moved C21 192.2 mm to (93.9, 60.7), turned to -90 degrees
- moved C20 188.4 mm to (80.8, 111.9)
- moved C3 187.2 mm to (80.0, 122.9)
- moved C1 149.8 mm to (125.5, 82.3), turned to 180 degrees
- moved TP13 122.0 mm to (148.8, 115.2)
- moved TP12 118.5 mm to (153.9, 115.2)
- moved Q3 40.2 mm to (65.6, 70.2)
- moved JP1 19.9 mm to (129.5, 79.8)
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Connections:
- C2 pad 2: /VCC_STRIP -> /VCC_STRIP1
- J8 pad 4: /VCC_STRIP -> /VCC_STRIP1

Commit message: PCB Design halfway
Parts:
- TP11, TP14, TP15, TP5: moved to B.Cu
- moved TP14 202.8 mm to (70.2, 71.5), turned to 180 degrees
- moved TP15 183.8 mm to (89.3, 73.3), turned to 180 degrees
- moved TP5 128.7 mm to (138.2, 66.0), turned to 180 degrees
- moved TP10 126.9 mm to (142.4, 83.6)
- moved R30 52.8 mm to (93.4, 65.2), turned to 180 degrees
- moved D1 16.1 mm to (89.7, 70.7)
- moved TP4 15.7 mm to (105.5, 65.3)
- moved TP3 11.1 mm to (138.2, 62.6)
- moved C7 10.7 mm to (127.1, 55.8), turned to 90 degrees
- moved C6 10.6 mm to (130.2, 55.8), turned to 90 degrees
- moved R11 10.5 mm to (131.7, 64.0), turned to 0 degrees
- moved C8 10.5 mm to (131.7, 65.7), turned to 180 degrees
- moved C5 9.38 mm to (128.7, 55.8), turned to 90 degrees
- moved C10 8.46 mm to (114.9, 55.5)
- moved R12 7.87 mm to (125.6, 56.3), turned to -90 degrees
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Connections:
- IC3 pad 12: +12V -> +3.3V
Routing:
- net GND: track 0.00 -> 89.6 mm, vias 0 -> 11
- net +3.3V: track 0.00 -> 87.0 mm, vias 0 -> 2
- net +5V: track 0.00 -> 72.4 mm, vias 0 -> 2
- net Net-(IC1-VSYS): track 0.00 -> 27.1 mm, vias 0 -> 1
- net /Regulator5V/VCC: track 0.00 -> 25.8 mm, vias 0 -> 2
- net Net-(U3-GPIO16): track 0.00 -> 19.0 mm
- net Net-(IC1-VBUS): track 0.00 -> 17.4 mm
- net +12V: track 0.00 -> 15.9 mm
- net Net-(C9-Pad1): track 0.00 -> 13.1 mm, vias 0 -> 2
- net /Regulator5V/SW: track 0.00 -> 10.2 mm, vias 0 -> 2
- net /Regulator5V/FB: track 0.00 -> 8.11 mm
- net Net-(D1-K): track 0.00 -> 7.14 mm
- net /Regulator5V/MODE: track 0.00 -> 5.79 mm
- net Net-(R31-Pad2): track 0.00 -> 5.45 mm
- net /Regulator5V/BST: track 0.00 -> 3.55 mm
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- added copper zone on F.Cu, net +12V
- added copper zone on F.Cu, net +3.3V
- added copper zone on F.Cu, net /Regulator5V/SW
- added copper zone on B.Cu, net GND
- added copper zone on F.Cu, net GND
Other:
- board size 113.2 x 85 mm -> 113 x 85 mm

Commit message: Nearly finished, just some DRC Errors te check
Parts:
- TP10, TP6, TP8, TP9: moved to B.Cu
- moved C16 22.1 mm to (120.8, 106.1), turned to 90 degrees
- moved TP14 21.9 mm to (91.8, 75.4)
- moved TP7 19.9 mm to (64.9, 91.5)
- moved TP6 19.7 mm to (61.8, 91.7), turned to 180 degrees
- moved TP11 17.4 mm to (49.4, 75.3)
- moved C18 6.00 mm to (101.3, 103.5), turned to 90 degrees
- moved TP10 2.16 mm to (142.2, 81.4), turned to 180 degrees
- moved C1 1.91 mm to (125.5, 80.4)
- moved C19 1.66 mm to (68.1, 113.3)
- moved J5 0.34 mm to (77.5, 127.6)
- moved C4 0.25 mm to (125.6, 64.0)
- moved C3 0.15 mm to (79.9, 122.9)
- turned TP8 to 180 degrees
- turned TP9 to 180 degrees
Connections:
- J2 pad 4: /Display_SDA -> /Display_MOSI
- J2 pad 5: /Display_SCL -> /Display_CLK
- J3 pad 4: /Display_SDA -> /Display_MOSI
- J3 pad 5: /Display_SCL -> /Display_CLK
Routing:
- net GND: track 89.6 -> 702.0 mm, vias 11 -> 32
- net +12V: track 15.9 -> 335.0 mm, vias 0 -> 14
- net +3.3V: track 87.0 -> 336.6 mm, vias 2 -> 9
- net +5V: track 72.4 -> 230.3 mm, vias 2 -> 8
- net /STOP_PIN2: track 0.00 -> 134.2 mm, vias 0 -> 2
- net /Display_CLK: track 0.00 -> 126.4 mm, vias 0 -> 5
- net /Display_MOSI: track 0.00 -> 115.8 mm, vias 0 -> 3
- net /STOP_PIN1: track 0.00 -> 108.5 mm
- net /Display_DC: track 0.00 -> 107.8 mm, vias 0 -> 2
- net /VCC_MUX: track 0.00 -> 103.4 mm, vias 0 -> 3
- net /TXD_PI4: track 0.00 -> 89.5 mm, vias 0 -> 11
- net /RXD_PI4: track 0.00 -> 88.2 mm, vias 0 -> 8
- net /Display_RES: track 0.00 -> 85.3 mm, vias 0 -> 4
- net /MUX_RX4: track 0.00 -> 76.9 mm, vias 0 -> 3
- net /MD2_STEP: track 0.00 -> 76.7 mm, vias 0 -> 5
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Other:
- board size 113 x 85 mm -> 113.1 x 85 mm

Commit message: Added name on PCB....
Other:
- board text added: "Project Healthbot PCB V0.1"
Changed lines of the file:
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@@
 		(layer "Edge.Cuts")
+	)
+	(gr_text "Project Healthbot PCB\nV0.1"
+		(at 154.175 98.725 90)
+		(layer "B.SilkS")
+		(effects
+			(font
+				(size 3 1.5)
+				(thickness 0.15)
+				(bold yes)
+			)
+			(justify left bottom mirror)
+		)
 	)
 	(gr_text "CAMERA\n"

Commit message: Finished!
Parts:
- added Logo: , clipboard:d0ed0aed-a5b7-4fbb-959d-d2596cb26e0d, F.Cu at (76.5, 70.0)
- TP12, TP13: moved to B.Cu
- moved C1 10.8 mm to (118.2, 88.4), turned to 0 degrees
- moved J15 1.78 mm to (153.4, 77.8)
- moved C6 1.08 mm to (131.2, 55.8)
- moved C4 0.95 mm to (124.7, 64.0)
- moved R27 0.94 mm to (151.7, 121.6)
- moved R25 0.69 mm to (136.7, 131.9)
- moved R24 0.69 mm to (147.1, 121.6)
- moved C5 0.55 mm to (129.2, 55.8)
- moved C2 0.38 mm to (68.2, 122.4)
- moved C3 0.30 mm to (80.1, 122.7)
- moved C22 0.27 mm to (138.2, 59.8)
- moved R31 0.27 mm to (134.7, 59.8)
- moved TP13 0.19 mm to (148.9, 115.0), turned to 180 degrees
- moved JP3 0.19 mm to (120.3, 116.4)
- moved C9 0.17 mm to (121.4, 53.5)
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Routing:
- net +3.3V: track 336.6 -> 475.7 mm, vias 9 -> 17
- net GND: track 702.0 -> 771.2 mm, vias 32 -> 37
- net +5V: track 230.3 -> 279.8 mm, vias 8 -> 13
- net /MUX_RX4: track 76.9 -> 63.9 mm
- net +12V: track 335.0 -> 329.5 mm
- net /MUX_TX3: track 66.0 -> 64.9 mm
- net /MUX_TX1: track 39.6 -> 40.5 mm
- net /VCC_MUX: track 103.4 -> 104.3 mm
- net Net-(J9-Pin_2): track 4.69 -> 5.42 mm
- net Net-(J10-Pin_2): track 5.79 -> 6.51 mm
- net Net-(J9-Pin_1): vias 0 -> 2
- net Net-(J10-Pin_1): vias 0 -> 2
- net /TXD_PI4: vias 11 -> 10
- net /MUX_RX2: vias 4 -> 3
- net /MD1_STEP: vias 5 -> 4
Other:
- board text added: "12V"
- board text added: "3.3V"
- board text added: "5V"
- board text added: "Extra"
- board text added: "GND"
- board text added: "GND RX3"
- board text added: "GND TX4"
- board text added: "LS1_VCC"
- board text added: "LS2_VCC"
- board text added: "MUX_UART"
- board text added: "PI4 Shutdown"
- board text added: "Project Healthbot V0.1"
- board text added: "RX4 VCC"
- board text added: "TX3 VCC"
- board text added: "x"
- board text removed: "Project Healthbot PCB V0.1"
