File: KiCAD_Proj/universalConnectorBoard.kicad_pcb (KiCad board)
At the start: 2 copper layers, 113.1 x 85 mm, 103 parts, among them IC1 RPI_Pico_EvaluationBoard, IC2 SN74LV4052ADR, IC3 TPS51397ARJER, IC4 TCA9534DWR, J1 691401700003B, J10 Cheeks, J11 MD_SW1, J12 MD_SW2, J13 Motor1, J14 Motor2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

Commit message: Final version
Parts:
- moved TP5 5.57 mm to (93.3, 69.4)
- moved PS1 1.32 mm to (97.9, 59.0)
- moved TP14 1.06 mm to (92.6, 76.1)
- moved D1 0.90 mm to (88.8, 70.7)
- moved TP4 0.13 mm to (105.5, 65.4)
- renumbered TP5 to TP1, TP15 to TP5
Routing:
- net +5V: track 279.8 -> 281.4 mm, vias 13 -> 14
- net +12V: track 329.5 -> 330.3 mm
- net GND: track 771.2 -> 771.7 mm
- removed copper zone on F.Cu, net +3.3V
