File: KiCAD_Proj/universalConnectorBoard.kicad_sch (KiCad schematic)
At the start: 71 parts, among them IC1 RPI_Pico_EvaluationBoard, IC2 SN74LV4052ADR, IC4 TCA9534DWR, J1 691401700003B, J10 Cheeks, J11 MD_SW1, J12 MD_SW2, J13 Motor1, J14 Motor2, J15 Extra VCC/GND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

Commit message: Final version
Parts:
- renumbered TP5 to TP1, TP15 to TP5
Changed lines of the file:
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@@
 		(on_board yes)
 		(dnp no)
-		(property "Reference" "TP15"
+		(property "Reference" "TP5"
 			(at 79.502 73.406 0)
 			(effects
@@
 			(project "universalConnectorBoard"
 				(path "/4d36baa7-ef48-416a-b1c8-6a662c0af28f"
-					(reference "TP15")
+					(reference "TP5")
 					(unit 1)
 				)
@@
 		(on_board yes)
 		(dnp no)
-		(property "Reference" "TP5"
+		(property "Reference" "TP1"
 			(at 232.156 50.546 90)
 			(effects
@@
 			(project "universalConnectorBoard"
 				(path "/4d36baa7-ef48-416a-b1c8-6a662c0af28f"
-					(reference "TP5")
+					(reference "TP1")
 					(unit 1)
 				)
